Commit message: update

File: urdf/cassie.urdf (robot description, URDF)
Before this commit: robot cassie, 18 links, 17 joints
Joints:
- joint hip_flexion_left: limit lower=-0.8727 upper=1.3963 effort=12.2 velocity=8.5085 -> lower=-0.8727 upper=1.3963 effort=18.75 velocity=251.2
- joint hip_flexion_right: limit lower=-0.8727 upper=1.3963 effort=12.2 velocity=8.5085 -> lower=-0.8727 upper=1.3963 effort=18.75 velocity=251.2
- joint knee_joint_left: limit lower=-2.8623 upper=-0.6458 effort=12.2 velocity=8.5085 -> lower=-2.8623 upper=-0.6458 effort=18.75 velocity=251.2
- joint knee_joint_right: limit lower=-2.8623 upper=-0.6458 effort=12.2 velocity=8.5085 -> lower=-2.8623 upper=-0.6458 effort=18.75 velocity=251.2
